File: Chessboard-Hardware-2.kicad_pcb (KiCad board)
At the start: 2 copper layers, 0 parts

Commit message: Setup for chessboard layout
Parts:
- added H1: MountingHole, MountingHole:MountingHole_2.7mm_M2.5, F.Cu at (54.0, 54.0)
- added H2: MountingHole, MountingHole:MountingHole_2.7mm_M2.5, F.Cu at (246.0, 54.0)
- added H3: MountingHole, MountingHole:MountingHole_2.7mm_M2.5, F.Cu at (246.0, 246.0)
- added H4: MountingHole, MountingHole:MountingHole_2.7mm_M2.5, F.Cu at (54.0, 246.0)
- added J1: Raspberry_Pi_0, Project Library:Raspberry_Pi_Zero_Socketed_THT_FaceDown_MountingHoles, F.Cu at (67.8, 93.6)
Other:
- board outline added: 200 x 200 mm
